File: PCB/HB-RC-4-Dis-TH.kicad_pcb (KiCad board)
At the start: 2 copper layers, 51 x 51 mm, 58 parts, among them J1 FTDI, J3 eInk, J4 ISP, J5 Power, Q1 IRLML6346TRBPF, SW1 T1, SW2 T2, SW3 T3, SW4 T4, SW5 Config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

Commit message: update pcb V2.1
Parts:
- moved R9 24.4 mm to (53.3, 31.5), turned to 180 degrees
- moved C1 0.23 mm to (17.1, 48.4)
- moved D2 0.08 mm to (44.1, 59.5)
- renumbered J1 to FTDI1, J4 to ISP1, LiPo to J6
Connections:
- J3 pad : (no net) -> GND
- U1 pad 34: Net-(U1-Pad34) -> /B_MEASURE
- U1 pad 37: /B_MEASURE -> Net-(U1-Pad37)
Routing:
- net GND: track 220.2 -> 175.4 mm, vias 48 -> 60
- net /B_MEASURE: track 48.3 -> 20.5 mm
- net +BATT: track 49.9 -> 68.7 mm
- net Net-(R2-Pad1): track 34.5 -> 51.9 mm
- net Net-(SW3-Pad1): track 69.5 -> 52.4 mm
- net Net-(SW5-Pad1): track 79.9 -> 63.4 mm, vias 0 -> 3
- net /RX: track 54.2 -> 66.0 mm
- net /PREVGL: track 42.2 -> 32.8 mm, vias 2 -> 1
- net /SCK: track 76.8 -> 68.6 mm
- net Net-(C11-Pad1): track 23.5 -> 16.5 mm
- net /MISO: track 42.9 -> 48.5 mm
- net /CC1101_GDO0: track 21.8 -> 26.9 mm, vias 1 -> 3
- net Net-(SW2-Pad1): track 26.1 -> 31.0 mm, vias 0 -> 2
- net /CC1101_CS: track 17.3 -> 20.5 mm
- net /TX: track 80.4 -> 83.4 mm
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Other:
- board text added: "V2.1"
- board text removed: "V2.0"

Commit message: update pcb
Parts:
- added R8-2: 1, Resistor_SMD:R_0805_2012Metric_Pad1.15x1.40mm_HandSolder, B.Cu at (51.5, 50.1)
- D6: value LED bl -> LED wt
- L1: value 100µH -> 68µH
- R12: value 240 -> 1k
- R7: value 2k2 -> 4k7
- R8: value 0.47 / 3.00 -> 1
Routing:
- net GND: track 175.4 -> 162.3 mm
- net /RESE: track 19.0 -> 19.6 mm
Changed lines of the file:
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@@
   (general
     (thickness 1.6)
-    (drawings 80)
-    (tracks 877)
+    (drawings 79)
+    (tracks 878)
     (zones 0)
-    (modules 58)
+    (modules 59)
     (nets 66)
   )
@@
     (add_net "Net-(U2-Pad6)")
   )
+  (module Resistor_SMD:R_0805_2012Metric_Pad1.15x1.40mm_HandSolder (layer B.Cu)
+    (at 51.53 50.07 180)
+    (descr "Resistor SMD 0805 (2012 Metric), square (rectangular) end terminal, IPC_7351 nominal with elongated pad for handsoldering. (Body size source: https://docs.google.com/spreadsheets/d/1BsfQQcO9C6DZCsRaXUlFlo91Tg2WpOkGARC1WS5S8t0/edit?usp=sharing), generated with kicad-footprint-generator")
+    (tags "resistor handsolder")
+    (attr smd)
+    (fp_text reference R8-2 (at 0 1.65) (layer B.SilkS) hide
+      (effects (font (size 1 1) (thickness 0.15)) (justify mirror))
+    )
+    (fp_text value 1 (at 0 -1.65) (layer B.Fab)
+      (effects (font (size 1 1) (thickness 0.15)) (justify mirror))
+    )
+    (fp_text user %R (at 0 0) (layer B.Fab)
+      (effects (font (size 0.5 0.5) (thickness 0.08)) (justify mirror))
+    )
+    (fp_line (start 1.85 -0.95) (end -1.85 -0.95) (layer B.CrtYd) (width 0.05))
+    (fp_line (start 1.85 0.95) (end 1.85 -0.95) (layer B.CrtYd) (width 0.05))
+    (fp_line (start -1.85 0.95) (end 1.85 0.95) (layer B.CrtYd) (width 0.05))
+    (fp_line (start -1.85 -0.95) (end -1.85 0.95) (layer B.CrtYd) (width 0.05))
+    (fp_line (start -0.261252 -0.71) (end 0.261252 -0.71) (layer B.SilkS) (width 0.12))
+    (fp_line (start -0.261252 0.71) (end 0.261252 0.71) (layer B.SilkS) (width 0.12))
+    (fp_line (start 1 -0.6) (end -1 -0.6) (layer B.Fab) (width 0.1))
+    (fp_line (start 1 0.6) (end 1 -0.6) (layer B.Fab) (width 0.1))
+    (fp_line (start -1 0.6) (end 1 0.6) (layer B.Fab) (width 0.1))
+    (fp_line (start -1 -0.6) (end -1 0.6) (layer B.Fab) (width 0.1))
+    (pad 2 smd roundrect (at 1.025 0 180) (size 1.15 1.4) (layers B.Cu B.Paste B.Mask) (roundrect_rratio 0.217391)
+      (net 3 GND))
+    (pad 1 smd roundrect (at -1.025 0 180) (size 1.15 1.4) (layers B.Cu B.Paste B.Mask) (roundrect_rratio 0.217391)
+      (net 51 /RESE))
+    (model ${KISYS3DMOD}/Resistor_SMD.3dshapes/R_0805_2012Metric.wrl
+      (at (xyz 0 0 0))
+      (scale (xyz 1 1 1))
+      (rotate (xyz 0 0 0))
+    )
+  )
   (module Package_SO:SO-4_4.4x3.6mm_P2.54mm (layer F.Cu)
     (at 48.76 19.08 180)
@@
       (effects (font (size 1 1) (thickness 0.15)) (justify mirror))
     )
-    (fp_text value 240 (at 0 -1.65) (layer B.Fab)
+    (fp_text value 1k (at 0 -1.65) (layer B.Fab)
       (effects (font (size 1 1) (thickness 0.15)) (justify mirror))
     )
@@
       (effects (font (size 1 1) (thickness 0.15)) (justify mirror))
     )
-    (fp_text value 2k2 (at 0 -1.65) (layer B.Fab)
+    (fp_text value 4k7 (at 0 -1.65) (layer B.Fab)
       (effects (font (size 1 1) (thickness 0.15)) (justify mirror))
     )
@@
       (effects (font (size 1 1) (thickness 0.15)))
     )
-    (fp_text value "LED bl" (at 0 1.65) (layer F.Fab)
+    (fp_text value "LED wt" (at 0 1.65) (layer F.Fab)
       (effects (font (size 1 1) (thickness 0.15)))
     )
@@
     (tags "resistor handsolder")
     (attr smd)
-    (fp_text reference R8 (at 0 1.65) (layer B.SilkS)
+    (fp_text reference R8 (at 2.77 1.08) (layer B.SilkS)
       (effects (font (size 1 1) (thickness 0.15)) (justify mirror))
     )
-    (fp_text value "0.47 / 3.00" (at 0 -1.65) (layer B.Fab)
+    (fp_text value 1 (at 0 -1.65) (layer B.Fab)
       (effects (font (size 1 1) (thickness 0.15)) (justify mirror))
     )
@@
       (effects (font (size 1 1) (thickness 0.15)) (justify mirror))
     )
-    (fp_text value 100µH (at 0 -3.2 90) (layer B.Fab)
+    (fp_text value 68µH (at 0 -3.2 90) (layer B.Fab)
       (effects (font (size 1 1) (thickness 0.15)) (justify mirror))
     )
@@
   (gr_line (start 25.54 50.03) (end 25.54 47.43) (layer F.SilkS) (width 0.12))
   (gr_line (start 31.94 52.73) (end 25.54 52.73) (layer F.SilkS) (width 0.12))
-  (gr_line (start 53.14 47.93) (end 53.14 52.73) (layer F.SilkS) (width 0.12))
   (gr_line (start 34.44 25.13) (end 53.14 25.13) (layer F.SilkS) (width 0.12))
   (gr_arc (start 18.84 40.88) (end 18.04 40.88) (angle -180) (layer Edge.Cuts) (width 0.05))
@@
   (gr_line (start 60.94 22.93) (end 60.94 54.93) (layer F.SilkS) (width 0.12))
   (gr_line (start 37.64 22.93) (end 60.94 22.93) (layer F.SilkS) (width 0.12))
-  (via (at 42.8 28.1) (size 0.8) (drill 0.4) (layers F.Cu B.Cu) (net 3))
   (segment (start 16.015 50.0297) (end 16.015 48.43) (width 0.25) (layer B.Cu) (net 1))
   (segment (start 16.015 50.0297) (end 16.015 51.165) (width 0.25) (layer B.Cu) (net 1))
@@
   (segment (start 25.3663 27.3037) (end 24.34 28.33) (width 0.25) (layer B.Cu) (net 2))
   (segment (start 42.99 19.0176) (end 42.99 19.5553) (width 0.25) (layer B.Cu) (net 2))
+  (via (at 42.8 28.1) (size 0.8) (drill 0.4) (layers F.Cu B.Cu) (net 3))
   (segment (start 42.9473 48.4341) (end 42.9473 48.9043) (width 0.25) (layer B.Cu) (net 3))
   (segment (start 43.0971 48.2843) (end 42.9473 48.4341) (width 0.25) (layer B.Cu) (net 3))
@@
   (segment (start 24.8651 29.8049) (end 26.34 28.33) (width 0.25) (layer B.Cu) (net 3))
   (segment (start 37.215 50.93) (end 37.215 48.73) (width 0.25) (layer B.Cu) (net 3))
-  (segment (start 49.3628 50.1277) (end 50.515 51.28) (width 0.25) (layer B.Cu) (net 3))
   (segment (start 50.515 51.28) (end 50.515 52.03) (width 0.25) (layer B.Cu) (net 3))
-  (segment (start 52.3652 44.8204) (end 52.3654 44.8206) (width 0.25) (layer B.Cu) (net 3))
-  (segment (start 52.3654 44.8206) (end 52.3654 47.1251) (width 0.25) (layer B.Cu) (net 3))
-  (segment (start 52.3654 47.1251) (end 49.3628 50.1277) (width 0.25) (layer B.Cu) (net 3))
   (segment (start 52.3652 44.8204) (end 52.3768 44.8088) (width 0.25) (layer B.Cu) (net 3))
   (segment (start 52.3768 44.8088) (end 52.3768 43.0605) (width 0.25) (layer B.Cu) (net 3))
@@
   (segment (start 45.6093 61.5146) (end 46.2647 62.17) (width 0.25) (layer F.Cu) (net 3))
   (segment (start 47.44 62.17) (end 46.2647 62.17) (width 0.25) (layer F.Cu) (net 3))
-  (segment (start 32.965 62.13) (end 26.3 62.13) (width 0.25) (layer F.Cu) (net 3))
-  (segment (start 26.3 62.13) (end 25.1247 62.13) (width 0.25) (layer F.Cu) (net 3))
-  (segment (start 24.3247 62.93) (end 25.1247 62.13) (width 0.25) (layer F.Cu) (net 3))
   (segment (start 28.74 51.23) (end 26.2 51.23) (width 0.25) (layer F.Cu) (net 3))
   (via (at 42.9473 48.4341) (size 0.8) (layers F.Cu B.Cu) (net 3))
@@
   (via (at 34.03 63.01) (size 0.8) (drill 0.4) (layers F.Cu B.Cu) (net 3))
   (via (at 46.05 45.26) (size 0.8) (drill 0.4) (layers F.Cu B.Cu) (net 3))
-  (via (at 51.98 50.31) (size 0.8) (drill 0.4) (layers F.Cu B.Cu) (net 3))
   (via (at 49.11 51.87) (size 0.8) (drill 0.4) (layers F.Cu B.Cu) (net 3))
   (via (at 63.24 45.48) (size 0.8) (drill 0.4) (layers F.Cu B.Cu) (net 3))
   (via (at 61.38 56.37) (size 0.8) (drill 0.4) (layers F.Cu B.Cu) (net 3))
+  (segment (start 50.515 51.28) (end 50.515 50.135) (width 0.25) (layer B.Cu) (net 3))
+  (via (at 55.79 49.36) (size 0.8) (drill 0.4) (layers F.Cu B.Cu) (net 3))
+  (segment (start 52.3652 44.8204) (end 52.3654 44.8206) (width 0.25) (layer B.Cu) (net 3))
+  (segment (start 52.3652 44.8204) (end 52.3652 47.6348) (width 0.25) (layer B.Cu) (net 3))
+  (segment (start 52.3652 47.6348) (end 52.3 47.7) (width 0.25) (layer B.Cu) (net 3))
   (segment (start 43.79 29.88) (end 43.79 30.9553) (width 0.25) (layer B.Cu) (net 4))
   (segment (start 43.79 30.9553) (end 43.7386 31.0067) (width 0.25) (layer B.Cu) (net 4))
@@
   (segment (start 51.39 43.68) (end 52.8934 43.68) (width 0.25) (layer F.Cu) (net 51))
   (segment (start 52.8934 43.68) (end 53.1255 43.4479) (width 0.25) (layer F.Cu) (net 51))
-  (segment (start 52.565 52.03) (end 53.1255 51.4695) (width 0.25) (layer B.Cu) (net 51))
-  (segment (start 53.1255 51.4695) (end 53.1255 43.4479) (width 0.25) (layer B.Cu) (net 51))
   (segment (start 58.3647 40.11) (end 58.3647 39.519) (width 0.25) (layer B.Cu) (net 51))
   (segment (start 58.3647 39.519) (end 58.1579 39.3122) (width 0.25) (layer B.Cu) (net 51))
@@
   (via (at 58.1579 39.3122) (size 0.8) (layers F.Cu B.Cu) (net 51))
   (via (at 53.1255 43.4479) (size 0.8) (layers F.Cu B.Cu) (net 51))
+  (segment (start 53.14 49) (end 53.1255 43.4479) (width 0.25) (layer B.Cu) (net 51))
+  (segment (start 53.14 50.06) (end 53.14 49) (width 0.25) (layer B.Cu) (net 51))
+  (segment (start 53.13 50.07) (end 53.14 50.06) (width 0.25) (layer B.Cu) (net 51))
+  (segment (start 52.555 50.07) (end 53.13 50.07) (width 0.25) (layer B.Cu) (net 51))
+  (segment (start 52.565 50.635) (end 53.13 50.07) (width 0.25) (layer B.Cu) (net 51))
+  (segment (start 52.565 52.03) (end 52.565 50.635) (width 0.25) (layer B.Cu) (net 51))
   (segment (start 37.84 35.93) (end 36.84 35.93) (width 0.25) (layer F.Cu) (net 54))
   (segment (start 60.4727 48.1148) (end 60.4727 40.1518) (width 0.25) (layer B.Cu) (net 55))

Commit message: update pcb
Parts:
- moved D6 0.47 mm to (46.2, 15.4)
Routing:
- net GND: track 162.3 -> 151.6 mm, vias 60 -> 81
- net Net-(D6-Pad1): track 5.77 -> 6.36 mm
Other:
- outline, holes or cut-outs redrawn

Commit message: update pcb
Parts:
- added RST: Reset, Button_Switch_SMD:SW_SPST_B3U-1000P, B.Cu at (15.9, 23.6)
- R1, R2: value 330 -> 240
Connections:
- J3 pad : GND -> (no net)
Routing:
- net /RESET: track 72.4 -> 87.8 mm
- net GND: vias 81 -> 80
Changed lines of the file:
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@@
     (thickness 1.6)
     (drawings 65)
-    (tracks 901)
+    (tracks 906)
     (zones 0)
-    (modules 59)
+    (modules 60)
     (nets 66)
   )
@@
     (add_net "Net-(U2-Pad6)")
   )
+  (module Button_Switch_SMD:SW_SPST_B3U-1000P (layer B.Cu)
+    (at 15.94 23.59 270)
+    (descr "Ultra-small-sized Tactile Switch with High Contact Reliability, Top-actuated Model, without Ground Terminal, without Boss")
+    (tags "Tactile Switch")
+    (attr smd)
+    (fp_text reference RST (at -1.54 -3.2 180) (layer B.SilkS)
+      (effects (font (size 1 1) (thickness 0.15)) (justify mirror))
+    )
+    (fp_text value Reset (at 0 -2.5 90) (layer B.Fab)
+      (effects (font (size 1 1) (thickness 0.15)) (justify mirror))
+    )
+    (fp_circle (center 0 0) (end 0.75 0) (layer B.Fab) (width 0.1))
+    (fp_line (start -1.5 -1.25) (end -1.5 1.25) (layer B.Fab) (width 0.1))
+    (fp_line (start 1.5 -1.25) (end -1.5 -1.25) (layer B.Fab) (width 0.1))
+    (fp_line (start 1.5 1.25) (end 1.5 -1.25) (layer B.Fab) (width 0.1))
+    (fp_line (start -1.5 1.25) (end 1.5 1.25) (layer B.Fab) (width 0.1))
+    (fp_line (start 1.65 1.4) (end 1.65 1.1) (layer B.SilkS) (width 0.12))
+    (fp_line (start -1.65 1.4) (end 1.65 1.4) (layer B.SilkS) (width 0.12))
+    (fp_line (start -1.65 1.1) (end -1.65 1.4) (layer B.SilkS) (width 0.12))
+    (fp_line (start 1.65 -1.4) (end 1.65 -1.1) (layer B.SilkS) (width 0.12))
+    (fp_line (start -1.65 -1.4) (end 1.65 -1.4) (layer B.SilkS) (width 0.12))
+    (fp_line (start -1.65 -1.1) (end -1.65 -1.4) (layer B.SilkS) (width 0.12))
+    (fp_line (start -2.4 1.65) (end -2.4 -1.65) (layer B.CrtYd) (width 0.05))
+    (fp_line (start 2.4 1.65) (end -2.4 1.65) (layer B.CrtYd) (width 0.05))
+    (fp_line (start 2.4 -1.65) (end 2.4 1.65) (layer B.CrtYd) (width 0.05))
+    (fp_line (start -2.4 -1.65) (end 2.4 -1.65) (layer B.CrtYd) (width 0.05))
+    (fp_text user %R (at 0 2.5 90) (layer B.Fab)
+      (effects (font (size 1 1) (thickness 0.15)) (justify mirror))
+    )
+    (pad 2 smd rect (at 1.7 0 270) (size 0.9 1.7) (layers B.Cu B.Paste B.Mask)
+      (net 2 /RESET))
+    (pad 1 smd rect (at -1.7 0 270) (size 0.9 1.7) (layers B.Cu B.Paste B.Mask)
+      (net 3 GND))
+    (model ${KISYS3DMOD}/Button_Switch_SMD.3dshapes/SW_SPST_B3U-1000P.wrl
+      (at (xyz 0 0 0))
+      (scale (xyz 1 1 1))
+      (rotate (xyz 0 0 0))
+    )
+  )
   (module Resistor_SMD:R_0805_2012Metric_Pad1.15x1.40mm_HandSolder (layer B.Cu)
     (at 51.53 50.07 180)
@@
       (net 49 "Net-(J3-Pad1)"))
     (pad "" smd rect (at 7.65 1.4 90) (size 1.8 4) (layers F.Cu F.Paste F.Mask))
-    (pad "" smd rect (at -7.65 1.4 90) (size 1.8 4) (layers F.Cu F.Paste F.Mask)
-      (net 3 GND))
+    (pad "" smd rect (at -7.65 1.4 90) (size 1.8 4) (layers F.Cu F.Paste F.Mask))
     (model ${KISYS3DMOD}/Connector_FFC-FPC.3dshapes/TE_2-84952-4_1x24-1MP_P1.0mm_Horizontal.wrl
       (at (xyz 0 0 0))
@@
       (effects (font (size 1 1) (thickness 0.15)) (justify mirror))
     )
-    (fp_text value 330 (at 0 -1.65 180) (layer B.Fab)
+    (fp_text value 240 (at 0 -1.65 180) (layer B.Fab)
       (effects (font (size 1 1) (thickness 0.15)) (justify mirror))
     )
@@
       (effects (font (size 1 1) (thickness 0.15)) (justify mirror))
     )
-    (fp_text value 330 (at 0 -1.65 180) (layer B.Fab)
+    (fp_text value 240 (at 0 -1.65 180) (layer B.Fab)
       (effects (font (size 1 1) (thickness 0.15)) (justify mirror))
     )
@@
   (gr_line (start 60.94 22.93) (end 60.94 54.93) (layer F.SilkS) (width 0.12))
   (gr_line (start 37.64 22.93) (end 60.94 22.93) (layer F.SilkS) (width 0.12))
-  (segment (start 44.48 14.09) (end 47.87 14.09) (width 0.25) (layer F.Cu) (net 3))
   (segment (start 16.015 50.0297) (end 16.015 48.43) (width 0.25) (layer B.Cu) (net 1))
   (segment (start 16.015 50.0297) (end 16.015 51.165) (width 0.25) (layer B.Cu) (net 1))
@@
   (segment (start 25.3663 27.3037) (end 24.34 28.33) (width 0.25) (layer B.Cu) (net 2))
   (segment (start 42.99 19.0176) (end 42.99 19.5553) (width 0.25) (layer B.Cu) (net 2))
+  (segment (start 15.705499 29.804609) (end 14.65 28.74911) (width 0.25) (layer B.Cu) (net 2))
+  (segment (start 22.865391 29.804609) (end 15.705499 29.804609) (width 0.25) (layer B.Cu) (net 2))
+  (segment (start 24.34 28.33) (end 22.865391 29.804609) (width 0.25) (layer B.Cu) (net 2))
+  (segment (start 14.65 25.48) (end 14.65 28.74911) (width 0.25) (layer B.Cu) (net 2))
+  (segment (start 14.84 25.29) (end 14.65 25.48) (width 0.25) (layer B.Cu) (net 2))
+  (segment (start 15.94 25.29) (end 14.84 25.29) (width 0.25) (layer B.Cu) (net 2))
+  (segment (start 44.48 14.09) (end 47.87 14.09) (width 0.25) (layer F.Cu) (net 3))
   (via (at 42.8 28.1) (size 0.8) (drill 0.4) (layers F.Cu B.Cu) (net 3))
   (segment (start 42.9473 48.4341) (end 42.9473 48.9043) (width 0.25) (layer B.Cu) (net 3))
@@
   (via (at 20 42.5) (size 0.8) (drill 0.4) (layers F.Cu B.Cu) (net 3))
   (via (at 31.69 14.79) (size 0.8) (drill 0.4) (layers F.Cu B.Cu) (net 3))
-  (via (at 15.82 23.43) (size 0.8) (drill 0.4) (layers F.Cu B.Cu) (net 3))
-  (via (at 21.85 22.18) (size 0.8) (drill 0.4) (layers F.Cu B.Cu) (net 3))
+  (via (at 18.69 15.84) (size 0.8) (drill 0.4) (layers F.Cu B.Cu) (net 3))
   (via (at 39.26 53.31) (size 0.8) (drill 0.4) (layers F.Cu B.Cu) (net 3))
   (segment (start 42.79 41.18) (end 41.8153 41.18) (width 0.25) (layer F.Cu) (net 3))

Commit message: update pcb
Parts:
- moved RST 6.82 mm to (18.7, 17.4)
Routing:
- net /RESET: track 87.8 -> 94.4 mm
- net GND: vias 80 -> 84
Changed lines of the file:
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@@
     (thickness 1.6)
     (drawings 65)
-    (tracks 906)
+    (tracks 910)
     (zones 0)
     (modules 60)
@@
   )
   (module Button_Switch_SMD:SW_SPST_B3U-1000P (layer B.Cu)
-    (at 15.94 23.59 270)
+    (at 18.69 17.35 270)
     (descr "Ultra-small-sized Tactile Switch with High Contact Reliability, Top-actuated Model, without Ground Terminal, without Boss")
     (tags "Tactile Switch")
     (attr smd)
-    (fp_text reference RST (at -1.54 -3.2 180) (layer B.SilkS)
+    (fp_text reference RST (at 3.2 -0.06 180) (layer B.SilkS)
       (effects (font (size 1 1) (thickness 0.15)) (justify mirror))
     )
@@
   (segment (start 25.3663 27.3037) (end 24.34 28.33) (width 0.25) (layer B.Cu) (net 2))
   (segment (start 42.99 19.0176) (end 42.99 19.5553) (width 0.25) (layer B.Cu) (net 2))
-  (segment (start 15.705499 29.804609) (end 14.65 28.74911) (width 0.25) (layer B.Cu) (net 2))
   (segment (start 22.865391 29.804609) (end 15.705499 29.804609) (width 0.25) (layer B.Cu) (net 2))
   (segment (start 24.34 28.33) (end 22.865391 29.804609) (width 0.25) (layer B.Cu) (net 2))
-  (segment (start 14.65 25.48) (end 14.65 28.74911) (width 0.25) (layer B.Cu) (net 2))
-  (segment (start 14.84 25.29) (end 14.65 25.48) (width 0.25) (layer B.Cu) (net 2))
-  (segment (start 15.94 25.29) (end 14.84 25.29) (width 0.25) (layer B.Cu) (net 2))
+  (segment (start 18.69 19.05) (end 18.69 23.90239) (width 0.25) (layer B.Cu) (net 2))
+  (segment (start 14.87029 28.9694) (end 15.705499 29.804609) (width 0.25) (layer B.Cu) (net 2))
+  (segment (start 14.87029 27.7221) (end 14.87029 28.9694) (width 0.25) (layer B.Cu) (net 2))
+  (segment (start 18.69 23.90239) (end 14.87029 27.7221) (width 0.25) (layer B.Cu) (net 2))
   (segment (start 44.48 14.09) (end 47.87 14.09) (width 0.25) (layer F.Cu) (net 3))
   (via (at 42.8 28.1) (size 0.8) (drill 0.4) (layers F.Cu B.Cu) (net 3))
@@
   (via (at 20 42.5) (size 0.8) (drill 0.4) (layers F.Cu B.Cu) (net 3))
   (via (at 31.69 14.79) (size 0.8) (drill 0.4) (layers F.Cu B.Cu) (net 3))
-  (via (at 18.69 15.84) (size 0.8) (drill 0.4) (layers F.Cu B.Cu) (net 3))
   (via (at 39.26 53.31) (size 0.8) (drill 0.4) (layers F.Cu B.Cu) (net 3))
   (segment (start 42.79 41.18) (end 41.8153 41.18) (width 0.25) (layer F.Cu) (net 3))
   (via (at 43.03 41.52) (size 0.8) (drill 0.4) (layers F.Cu B.Cu) (net 3))
+  (via (at 20.22 22.52) (size 0.8) (drill 0.4) (layers F.Cu B.Cu) (net 3))
+  (via (at 14.88 25.48) (size 0.8) (drill 0.4) (layers F.Cu B.Cu) (net 3))
+  (via (at 17.16 23.18) (size 0.8) (drill 0.4) (layers F.Cu B.Cu) (net 3))
+  (via (at 27.68 17.84) (size 0.8) (drill 0.4) (layers F.Cu B.Cu) (net 3))
+  (via (at 45.12 52.47) (size 0.8) (drill 0.4) (layers F.Cu B.Cu) (net 3))
   (segment (start 43.79 29.88) (end 43.79 30.9553) (width 0.25) (layer B.Cu) (net 4))
   (segment (start 43.79 30.9553) (end 43.7386 31.0067) (width 0.25) (layer B.Cu) (net 4))
