File: PCB/HB-RC-4-Dis-TH.sch (KiCad schematic (older format))
At the start: 59 parts, among them J3 eInk, J5 Power, J6 Batt, Q1 IRLML6346TRBPF, SW1 T1, SW2 T2, SW3 T3, SW4 T4, SW5 Config, U1 ATmega1284P-AU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

Commit message: update pcb
Parts:
- R1, R2: value 330 -> 240
Changed lines of the file:
@@
 P 8850 2750
 F 0 "R1" V 8880 2580 50  0000 C CNN
-F 1 "330" V 8840 2750 50  0000 C CNN
+F 1 "240" V 8840 2750 50  0000 C CNN
 F 2 "Resistor_SMD:R_0805_2012Metric_Pad1.15x1.40mm_HandSolder" V 8780 2750 50  0001 C CNN
 F 3 "~" H 8850 2750 50  0001 C CNN
@@
 P 8850 2850
 F 0 "R2" V 8880 2680 50  0000 C CNN
-F 1 "330" V 8840 2850 50  0000 C CNN
+F 1 "240" V 8840 2850 50  0000 C CNN
 F 2 "Resistor_SMD:R_0805_2012Metric_Pad1.15x1.40mm_HandSolder" V 8780 2850 50  0001 C CNN
 F 3 "~" H 8850 2850 50  0001 C CNN

Commit message: update pcb
Parts:
- added RST: Reset, Button_Switch_SMD:SW_SPST_B3U-1000P, symbol Switch:SW_Push
Connections:
- net GND: now also RST.1
- net RESET: now also RST.2
Changed lines of the file:
@@
 Wire Wire Line
 	4470 5750 4470 5870
+$Comp
+L Switch:SW_Push RST
+U 1 1 5F7BB12C
+P 6020 2760
+F 0 "RST" H 6020 3045 50  0000 C CNN
+F 1 "Reset" H 6020 2954 50  0000 C CNN
+F 2 "Button_Switch_SMD:SW_SPST_B3U-1000P" H 6020 2960 50  0001 C CNN
+F 3 "~" H 6020 2960 50  0001 C CNN
+	1    6020 2760
+	1    0    0    -1
+$EndComp
+Text Label 6220 2760 0    50   ~ 0
+RESET
+$Comp
+L power:GND #PWR0103
+U 1 1 5F7BC17D
+P 5820 2760
+F 0 "#PWR0103" H 5820 2510 50  0001 C CNN
+F 1 "GND" H 5825 2587 50  0000 C CNN
+F 2 "" H 5820 2760 50  0001 C CNN
+F 3 "" H 5820 2760 50  0001 C CNN
+	1    5820 2760
+	1    0    0    -1
+$EndComp
 $EndSCHEMATC

Commit message: replaced 3.3V LDO with 3.0V
Parts:
- U3: value MCP1703T-3302E/CB -> MCP 1700T-3002E
Connections:
- net labels added: +3V0
- net labels removed: +3.3V
Changed lines of the file:
@@
 $EndComp
 $Comp
-L power:+3.3V #PWR010
+L power:+3V0 #PWR010
 U 1 1 5F2DB7AA
 P 9380 830
 F 0 "#PWR010" H 9380 680 50  0001 C CNN
-F 1 "+3.3V" H 9395 1003 50  0000 C CNN
+F 1 "+3V0" H 9395 1003 50  0000 C CNN
 F 2 "" H 9380 830 50  0001 C CNN
 F 3 "" H 9380 830 50  0001 C CNN
@@
 Connection ~ 7850 5630
 $Comp
-L power:+3.3V #PWR03
+L power:+3V0 #PWR03
 U 1 1 5F2F87CF
 P 7900 1220
 F 0 "#PWR03" H 7900 1070 50  0001 C CNN
-F 1 "+3.3V" H 7915 1393 50  0000 C CNN
+F 1 "+3V0" H 7915 1393 50  0000 C CNN
 F 2 "" H 7900 1220 50  0001 C CNN
 F 3 "" H 7900 1220 50  0001 C CNN
@@
 	890  1150 890  1000
 $Comp
-L power:+3.3V #PWR08
+L power:+3V0 #PWR08
 U 1 1 5F310749
 P 890 1000
 F 0 "#PWR08" H 890 850 50  0001 C CNN
-F 1 "+3.3V" H 905 1173 50  0000 C CNN
+F 1 "+3V0" H 905 1173 50  0000 C CNN
 F 2 "" H 890 1000 50  0001 C CNN
 F 3 "" H 890 1000 50  0001 C CNN
@@
 	8820 3650 8820 3600
 $Comp
-L power:+3.3V #PWR04
+L power:+3V0 #PWR04
 U 1 1 5F3152CF
 P 9010 3190
 F 0 "#PWR04" H 9010 3040 50  0001 C CNN
-F 1 "+3.3V" H 9025 3363 50  0000 C CNN
+F 1 "+3V0" H 9025 3363 50  0000 C CNN
 F 2 "" H 9010 3190 50  0001 C CNN
 F 3 "" H 9010 3190 50  0001 C CNN
@@
 	2040 1360 2460 1360
 $Comp
-L power:+3.3V #PWR02
+L power:+3V0 #PWR02
 U 1 1 5F308BC9
 P 2460 1260
 F 0 "#PWR02" H 2460 1110 50  0001 C CNN
-F 1 "+3.3V" H 2475 1433 50  0000 C CNN
+F 1 "+3V0" H 2475 1433 50  0000 C CNN
 F 2 "" H 2460 1260 50  0001 C CNN
 F 3 "" H 2460 1260 50  0001 C CNN
@@
 MISO
 $Comp
-L power:+3.3V #PWR013
+L power:+3V0 #PWR013
 U 1 1 5F34FA00
 P 3370 1100
 F 0 "#PWR013" H 3370 950 50  0001 C CNN
-F 1 "+3.3V" H 3385 1273 50  0000 C CNN
+F 1 "+3V0" H 3385 1273 50  0000 C CNN
 F 2 "" H 3370 1100 50  0001 C CNN
 F 3 "" H 3370 1100 50  0001 C CNN
@@
 	4470 2960 4470 3160
 $Comp
-L power:+3.3V #PWR06
+L power:+3V0 #PWR06
 U 1 1 5F3C27F2
 P 3050 2250
 F 0 "#PWR06" H 3050 2100 50  0001 C CNN
-F 1 "+3.3V" H 3065 2423 50  0000 C CNN
+F 1 "+3V0" H 3065 2423 50  0000 C CNN
 F 2 "" H 3050 2250 50  0001 C CNN
 F 3 "" H 3050 2250 50  0001 C CNN
@@
 $EndComp
 $Comp
-L power:+3.3V #PWR024
+L power:+3V0 #PWR024
 U 1 1 5F3EC9C8
 P 4470 4590
 F 0 "#PWR024" H 4470 4440 50  0001 C CNN
-F 1 "+3.3V" H 4485 4763 50  0000 C CNN
+F 1 "+3V0" H 4485 4763 50  0000 C CNN
 F 2 "" H 4470 4590 50  0001 C CNN
 F 3 "" H 4470 4590 50  0001 C CNN
@@
 $EndComp
 $Comp
-L power:+3.3V #PWR0101
+L power:+3V0 #PWR0101
 U 1 1 5F3C06CE
 P 1610 3730
 F 0 "#PWR0101" H 1610 3580 50  0001 C CNN
-F 1 "+3.3V" H 1440 3780 50  0000 C CNN
+F 1 "+3V0" H 1440 3780 50  0000 C CNN
 F 2 "" H 1610 3730 50  0001 C CNN
 F 3 "" H 1610 3730 50  0001 C CNN
@@
 $EndComp
 $Comp
-L power:+3.3V #PWR029
+L power:+3V0 #PWR029
 U 1 1 5F3ED0ED
 P 2610 7010
 F 0 "#PWR029" H 2610 6860 50  0001 C CNN
-F 1 "+3.3V" H 2625 7183 50  0000 C CNN
+F 1 "+3V0" H 2625 7183 50  0000 C CNN
 F 2 "" H 2610 7010 50  0001 C CNN
 F 3 "" H 2610 7010 50  0001 C CNN
@@
 $EndComp
 $Comp
-L power:+3.3V #PWR033
+L power:+3V0 #PWR033
 U 1 1 5F3ACF13
 P 3430 7010
 F 0 "#PWR033" H 3430 6860 50  0001 C CNN
-F 1 "+3.3V" H 3445 7183 50  0000 C CNN
+F 1 "+3V0" H 3445 7183 50  0000 C CNN
 F 2 "" H 3430 7010 50  0001 C CNN
 F 3 "" H 3430 7010 50  0001 C CNN
@@
 $EndComp
 $Comp
-L power:+3.3V #PWR031
+L power:+3V0 #PWR031
 U 1 1 5F3B2D50
 P 3020 7010
 F 0 "#PWR031" H 3020 6860 50  0001 C CNN
-F 1 "+3.3V" H 3035 7183 50  0000 C CNN
+F 1 "+3V0" H 3035 7183 50  0000 C CNN
 F 2 "" H 3020 7010 50  0001 C CNN
 F 3 "" H 3020 7010 50  0001 C CNN
@@
 $EndComp
 $Comp
-L power:+3.3V #PWR035
+L power:+3V0 #PWR035
 U 1 1 5F3B35D6
 P 3830 7010
 F 0 "#PWR035" H 3830 6860 50  0001 C CNN
-F 1 "+3.3V" H 3845 7183 50  0000 C CNN
+F 1 "+3V0" H 3845 7183 50  0000 C CNN
 F 2 "" H 3830 7010 50  0001 C CNN
 F 3 "" H 3830 7010 50  0001 C CNN
@@
 $EndComp
 $Comp
-L power:+3.3V #PWR037
+L power:+3V0 #PWR037
 U 1 1 5F3B3C06
 P 4220 7010
 F 0 "#PWR037" H 4220 6860 50  0001 C CNN
-F 1 "+3.3V" H 4235 7183 50  0000 C CNN
+F 1 "+3V0" H 4235 7183 50  0000 C CNN
 F 2 "" H 4220 7010 50  0001 C CNN
 F 3 "" H 4220 7010 50  0001 C CNN
@@
 P 2660 5750
 F 0 "U3" H 2660 5770 50  0000 C CNN
-F 1 "MCP1703T-3302E/CB" H 2700 5860 50  0000 C CNN
+F 1 "MCP 1700T-3002E" H 2700 5860 50  0000 C CNN
 F 2 "Package_TO_SOT_SMD:SOT-23" H 2660 5950 50  0001 C CNN
 F 3 "http://ww1.microchip.com/downloads/en/DeviceDoc/20005122B.pdf" H 2660 5700 50  0001 C CNN
@@
 $EndComp
 $Comp
-L power:+3.3V #PWR046
+L power:+3V0 #PWR046
 U 1 1 5F5F1E01
 P 3140 5540
 F 0 "#PWR046" H 3140 5390 50  0001 C CNN
-F 1 "+3.3V" H 3270 5550 50  0000 C CNN
+F 1 "+3V0" H 3270 5550 50  0000 C CNN
 F 2 "" H 3140 5540 50  0001 C CNN
 F 3 "" H 3140 5540 50  0001 C CNN
@@
 	2110 4810 2110 5750
 $Comp
-L power:+3.3V #PWR047
+L power:+3V0 #PWR047
 U 1 1 5F633211
 P 3210 4090
 F 0 "#PWR047" H 3210 3940 50  0001 C CNN
-F 1 "+3.3V" H 3040 4140 50  0000 C CNN
+F 1 "+3V0" H 3040 4140 50  0000 C CNN
 F 2 "" H 3210 4090 50  0001 C CNN
 F 3 "" H 3210 4090 50  0001 C CNN
